File: hardware/kitting_board.brd (EAGLE design)
At the start: 254 x 76.2 mm, 39 parts

Commit message: Added parts, completed traces
Added silkscreen
Parts:
- added J15, J16, J19: USB_A, USB_A_female_VRT:USB-A-H-FEMALE-VRT-PTH
- added J17, J18, J20: (no value), SparkFun-Connectors:USB-MICROB
- added JP10, JP8, JP9: JUMPER-SMT_2_NC_PASTE_SILK, SparkFun-Jumpers:SMT-JUMPER_2_NC_PASTE_SILK
- added LED10, LED8, LED9: (no value), adafruit:CHIPLED_0805
- added R10, R8, R9: (no value), adafruit:R0805
- moved JP6 0.25 mm to (166.1, 68.6)
Connections:
- new net D+10: J19.D+, J20.D+
- new net D+8: J15.D+, J18.D+
- new net D+9: J16.D+, J17.D+
- new net D-10: J19.D-, J20.D-
- new net D-8: J15.D-, J18.D-
- new net D-9: J16.D-, J17.D-
- new net N$15: LED8.A, R8.1
- new net N$16: JP8.1, R8.2
- new net N$17: LED9.A, R9.1
- new net N$18: JP9.1, R9.2
- new net N$19: LED10.A, R10.1
- new net N$20: JP10.1, R10.2
- new net VCC10: J19.VBUS, J20.VBUS, JP10.2
- new net VCC8: J15.VBUS, J18.VBUS, JP8.2
- new net VCC9: J16.VBUS, J17.VBUS, JP9.2
- net GND: now also J15.GND, J16.GND, J17.GND, J18.GND, J19.GND, J20.GND, LED10.C, LED8.C, LED9.C
Routing:
- net VCC10: track 0.00 -> 72.0 mm
- net VCC9: track 0.00 -> 72.0 mm
- net VCC8: track 0.00 -> 72.0 mm
- net D+8: track 0.00 -> 42.1 mm
- net D+9: track 0.00 -> 42.1 mm
- net D+10: track 0.00 -> 42.1 mm
- net D-10: track 0.00 -> 39.9 mm
- net D-9: track 0.00 -> 39.9 mm
- net D-8: track 0.00 -> 39.9 mm
- net N$19: track 0.00 -> 2.56 mm
- net N$17: track 0.00 -> 2.56 mm
- net N$15: track 0.00 -> 2.56 mm
- net N$20: track 0.00 -> 2.52 mm
- net N$18: track 0.00 -> 2.52 mm
- net N$16: track 0.00 -> 2.52 mm
Other:
- board text added: "2017.6.6"
- board text added: "Designed by Akram Ali"
- board text added: "KITTING SYSTEM"
- board text added: "SD card (firmware)"
- board text added: "Touchstone"
- board text added: "USB Gateway"
- board text added: "crtlabs.org"
- board text added: "v1.0"
