File: hardware/kitting_board.sch (EAGLE design)
At the start: 39 parts

Commit message: Added parts, completed traces
Added silkscreen
Parts:
- added J15, J16, J19: USB_A, USB_A_female_VRT:USB_A
- added J17, J18, J20: (no value), SparkFun-Connectors:USB_MICRO-B_SMT
- added JP10, JP8, JP9: JUMPER-SMT_2_NC_PASTE_SILK, SparkFun-Jumpers:JUMPER-SMT_2_NC_PASTE_SILK
- added LED10, LED8, LED9: (no value), adafruit:LEDCHIPLED_0805
- added R10, R8, R9: (no value), adafruit:R-US_R0805
Connections:
- new net D+10: J19.D+, J20.D+
- new net D+8: J15.D+, J18.D+
- new net D+9: J16.D+, J17.D+
- new net D-10: J19.D-, J20.D-
- new net D-8: J15.D-, J18.D-
- new net D-9: J16.D-, J17.D-
- new net N$15: LED8.A, R8.1
- new net N$16: JP8.1, R8.2
- new net N$17: LED9.A, R9.1
- new net N$18: JP9.1, R9.2
- new net N$19: LED10.A, R10.1
- new net N$20: JP10.1, R10.2
- new net VCC10: J19.VBUS, J20.VBUS, JP10.2
- new net VCC8: J15.VBUS, J18.VBUS, JP8.2
- new net VCC9: J16.VBUS, J17.VBUS, JP9.2
- net GND: now also J15.GND, J16.GND, J17.GND, J18.GND, J19.GND, J20.GND, LED10.C, LED8.C, LED9.C
